Commit message: fix the urdf file to fit the new package name

File: dofbot_digital/urdf/dofbot.urdf (robot description, URDF)
Before this commit: robot arm, 6 links, 5 joints
Links:
- link base_link: geometry collision mesh filename=package://dofbot_digital/meshes/base_link.STL; visual mesh filename=package://dofbot_digital/meshes/base_link.STL
- link link1: geometry collision mesh filename=package://dofbot_digital/meshes/link1.STL; visual mesh filename=package://dofbot_digital/meshes/link1.STL
- link link2: geometry collision mesh filename=package://dofbot_digital/meshes/link2.STL; visual mesh filename=package://dofbot_digital/meshes/link2.STL
- link link3: geometry collision mesh filename=package://dofbot_digital/meshes/link3.STL; visual mesh filename=package://dofbot_digital/meshes/link3.STL
- link link4: geometry collision mesh filename=package://dofbot_digital/meshes/link4.STL; visual mesh filename=package://dofbot_digital/meshes/link4.STL
- link link5: geometry collision mesh filename=package://dofbot_digital/meshes/link5.STL; visual mesh filename=package://dofbot_digital/meshes/link5.STL

Commit message: dofbot with gripper digital model description

File: dofbot_digital/urdf/dofbot.urdf (robot description, URDF)
Before this commit: robot arm, 6 links, 5 joints
Links:
- removed link link1
- removed link link2
- removed link link3
- removed link link4
- removed link link5
- added link arm_link1, mass 0.0279545499871709; collision mesh filename=package://dofbot_digital/meshes/X3plus/collision/arm_link1.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; visual mesh filename=package://dofbot_digital/meshes/X3plus/visual/arm_link1.STL
- added link arm_link2, mass 0.031605; collision mesh filename=package://dofbot_digital/meshes/X3plus/collision/arm_link2.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; visual mesh filename=package://dofbot_digital/meshes/X3plus/visual/arm_link2.STL
- added link arm_link3, mass 0.031605; collision mesh filename=package://dofbot_digital/meshes/X3plus/collision/arm_link3.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; visual mesh filename=package://dofbot_digital/meshes/X3plus/visual/arm_link3.STL
- added link arm_link4, mass 0.049766; collision mesh filename=package://dofbot_digital/meshes/X3plus/collision/arm_link4.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; visual mesh filename=package://dofbot_digital/meshes/X3plus/visual/arm_link4.STL
- added link arm_link5, mass 0.04069; collision mesh filename=package://dofbot_digital/meshes/X3plus/collision/arm_link5.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; visual mesh filename=package://dofbot_digital/meshes/X3plus/visual/arm_link5.STL
- added link llink1, mass 0.00121010771282268; collision mesh filename=package://dofbot_digital/meshes/X3plus/visual/llink1.STL; visual mesh filename=package://dofbot_digital/meshes/X3plus/visual/llink1.STL
- added link llink2, mass 0.0024469; collision mesh filename=package://dofbot_digital/meshes/X3plus/visual/llink2.STL; visual mesh filename=package://dofbot_digital/meshes/X3plus/visual/llink2.STL
- added link llink3, mass 0.00087627; collision mesh filename=package://dofbot_digital/meshes/X3plus/visual/llink3.STL; visual mesh filename=package://dofbot_digital/meshes/X3plus/visual/llink3.STL
- added link rlink1, mass 0.00117883201961805; collision mesh filename=package://dofbot_digital/meshes/X3plus/visual/rlink1.STL; visual mesh filename=package://dofbot_digital/meshes/X3plus/visual/rlink1.STL
- added link rlink2, mass 0.0024469; collision mesh filename=package://dofbot_digital/meshes/X3plus/visual/rlink2.STL; visual mesh filename=package://dofbot_digital/meshes/X3plus/visual/rlink2.STL
- added link rlink3, mass 0.00087627; collision mesh filename=package://dofbot_digital/meshes/X3plus/visual/rlink3.STL; visual mesh filename=package://dofbot_digital/meshes/X3plus/visual/rlink3.STL
Joints:
- removed joint joint1
- removed joint joint2
- removed joint joint3
- removed joint joint4
- removed joint joint5
- added joint arm_joint1: type revolute, parent base_link, child arm_link1, origin xyz=0 0 0.06605 rpy=-0.010805 0 1.5, axis 0 0 1, limit lower=-1.5708 upper=1.5708 effort=30 velocity=1.0
- added joint arm_joint2: type revolute, parent arm_link1, child arm_link2, origin xyz=0 0 0.0405 rpy=-1.5708 0 0, axis 0 0 -1, limit lower=-1.5708 upper=1.5708 effort=100 velocity=1
- added joint arm_joint3: type revolute, parent arm_link2, child arm_link3, origin xyz=0 -0.0829 0 rpy=0 0 0, axis 0 0 -1, limit lower=-1.5708 upper=1.5708 effort=100 velocity=1
- added joint arm_joint4: type revolute, parent arm_link3, child arm_link4, origin xyz=0 -0.0829 0 rpy=0 0 0, axis 0 0 -1, limit lower=-1.5708 upper=1.5708 effort=100 velocity=1
- added joint arm_joint5: type revolute, parent arm_link4, child arm_link5, origin xyz=-0.00215 -0.17455 0 rpy=1.5708 0 0, axis 0 0 1, limit lower=-1.5708 upper=3.14159 effort=100 velocity=1
- added joint grip_joint: type revolute, parent arm_link5, child rlink1, origin xyz=-0.0035 -0.012625 -0.0685 rpy=0 -1.5708 0, axis 0 0 1, limit lower=-1.54 upper=0 effort=100 velocity=1
- added joint llink_joint1: type continuous, parent arm_link5, child llink1, origin xyz=-0.0035 0.012375 -0.0685 rpy=0 -1.5708 0, axis 0 0 1, mimic joint=grip_joint multiplier=-1
- added joint llink_joint2: type continuous, parent llink1, child llink2, origin xyz=0.03 0.00065104 0 rpy=0 0 0, axis 0 0 1, mimic joint=grip_joint multiplier=1
- added joint llink_joint3: type continuous, parent arm_link5, child llink3, origin xyz=-0.0035 0.0045 -0.0505 rpy=0 -1.5708 0, axis 0 0 1, mimic joint=grip_joint multiplier=-1
- added joint rlink_joint2: type continuous, parent rlink1, child rlink2, origin xyz=0.03 -0.00075429 0 rpy=0 0 0, axis 0 0 1, mimic joint=grip_joint multiplier=-1
- added joint rlink_joint3: type continuous, parent arm_link5, child rlink3, origin xyz=-0.0035 -0.0045 -0.0505 rpy=0 -1.5708 0, axis 0 0 1, mimic joint=grip_joint multiplier=1
